File: hardware/esp32-polargraph.kicad_pcb (KiCad board)
At the start: 2 copper layers, 9.2 x 6.5 mm, 53 parts, among them J1 24VDC, J2 USB_C_Receptacle_USB2.0, J3 SSD1306, J4 Left motor, J5 Right motor, J6 Stepper A, J7 Stepper B, J8 Stepper C, SW1 BOOT, SW2 EN, U1 TMC2224-LA-T, U2 ESP32-S3-MINI-1, U3 NCP1117-3.3_SOT223, U4 TMC2224-LA-T

Commit message: Almost finished pcb
Parts:
- removed J3: SSD1306, Connector_PinHeader_2.54mm:PinHeader_1x04_P2.54mm_Vertical
- added 24V1: TestPoint, TestPoint:TestPoint_Pad_D2.0mm, F.Cu at (139.3, 81.6)
- added 3.3V1: TestPoint, TestPoint:TestPoint_Pad_D2.0mm, F.Cu at (133.8, 89.2)
- added 5V1: TestPoint, TestPoint:TestPoint_Pad_D2.0mm, F.Cu at (151.3, 115.9)
- added C20: 0.1uF, Capacitor_SMD:C_0603_1608Metric, F.Cu at (144.4, 102.5)
- added C21: 22uF, Capacitor_SMD:CP_Elec_4x5.4, F.Cu at (150.7, 107.7)
- added J9: Micro_SD_Card, Connector_Card:microSD_HC_Wuerth_693072010801, F.Cu at (79.0, 82.2)
- added R13: 4k7, Resistor_SMD:R_0603_1608Metric, F.Cu at (90.2, 98.2)
- added R14: 4k7, Resistor_SMD:R_0603_1608Metric, F.Cu at (87.8, 98.2)
- added R15: 1M, Resistor_SMD:R_0603_1608Metric, F.Cu at (81.5, 70.8)
- added R16: 10k, Resistor_SMD:R_0603_1608Metric, F.Cu at (90.5, 80.5)
- added R17: 10k, Resistor_SMD:R_0603_1608Metric, F.Cu at (88.8, 81.4)
- added R18: 10k, Resistor_SMD:R_0603_1608Metric, F.Cu at (89.0, 85.2)
- added U5: NCV4274ADT50RKG, Package_TO_SOT_SMD:TO-252-3_TabPin4, F.Cu at (149.5, 97.0)
- added U6: 0.96_SSD1306, polygraph:0.96_SSD1306, F.Cu at (72.3, 119.3)
- C11, C12: footprint Capacitor_SMD:CP_Elec_10x10.5 -> Capacitor_SMD:CP_Elec_4x5.4
- moved H4 104.1 mm to (151.4, 137.8), turned to -90 degrees
- moved H2 88.1 mm to (151.4, 68.8), turned to -90 degrees
- moved H1 84.3 mm to (76.5, 137.8), turned to -90 degrees
- moved J4 79.8 mm to (129.2, 123.4), turned to -90 degrees
- moved R3 79.5 mm to (120.0, 118.8), turned to 135 degrees
- moved R4 74.3 mm to (120.4, 111.0), turned to -135 degrees
- moved U1 71.0 mm to (112.9, 114.3), turned to -90 degrees
- moved C11 67.3 mm to (141.2, 71.0), turned to 90 degrees
- moved J1 66.6 mm to (144.0, 80.5), turned to 90 degrees
- moved JP2 66.4 mm to (105.2, 115.5), turned to 90 degrees
- moved C9 65.5 mm to (113.2, 110.1), turned to 0 degrees
- moved JP1 65.1 mm to (105.2, 111.8), turned to -90 degrees
- moved C6 65.0 mm to (116.8, 119.0), turned to -90 degrees
- moved C10 65.0 mm to (108.6, 111.2), turned to 90 degrees
- moved J6 64.3 mm to (94.1, 123.4), turned to -90 degrees
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Connections:
- J1 pad 1: +24V -> GND
- J1 pad 2: GND -> +24V
- J2 pad S1: GND -> Net-(J2-PadS1)
- J6 pad 2: +3V3 -> +5V
- J7 pad 2: +3V3 -> +5V
- J8 pad 2: +3V3 -> +5V
- U1 pad 29: (no net) -> GND
- U2 pad 12: Stepper A -> SPI_MISO
- U2 pad 13: Stepper B -> SPI_MOSI
- U2 pad 14: Stepper C -> SPI_CLK
- U2 pad 15: unconnected-(U2-Pad15) -> SPI_CS
- U2 pad 16: unconnected-(U2-Pad16) -> Net-(R14-Pad1)
- U2 pad 17: unconnected-(U2-Pad17) -> Net-(R13-Pad1)
- U2 pad 25: unconnected-(U2-Pad25) -> Stepper A
- U2 pad 26: unconnected-(U2-Pad26) -> Stepper B
- U2 pad 27: unconnected-(U2-Pad27) -> Stepper C
- U4 pad 29: (no net) -> GND
Routing:
- net +3V3: track 0.00 -> 244.8 mm, vias 0 -> 9
- net +5V: track 0.00 -> 131.5 mm
- net +24V: track 0.00 -> 127.0 mm, vias 0 -> 4
- net Stepper C: track 0.00 -> 67.4 mm, vias 0 -> 2
- net Stepper A: track 0.00 -> 62.4 mm, vias 0 -> 2
- net Stepper B: track 0.00 -> 58.3 mm, vias 0 -> 2
- net Net-(R10-Pad2): track 0.00 -> 49.3 mm, vias 0 -> 2
- net Net-(R9-Pad2): track 0.00 -> 46.2 mm, vias 0 -> 2
- net GND: track 0.00 -> 42.6 mm, vias 0 -> 4
- net SPI_MISO: track 0.00 -> 37.6 mm
- net SPI_CLK: track 0.00 -> 37.3 mm, vias 0 -> 2
- net Net-(C2-Pad2): track 0.00 -> 37.2 mm, vias 0 -> 2
- net SPI_MOSI: track 0.00 -> 37.2 mm
- net Net-(R5-Pad1): track 0.00 -> 36.8 mm, vias 0 -> 2
- net SPI_CS: track 0.00 -> 36.7 mm
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- added copper zone on B.Cu, net GND
- added copper zone on F.Cu, net GND
Other:
- board size 9.2 x 6.5 mm -> 85 x 79 mm
- board text added: "24VDC Tip +"
- board text added: "Made with <3 at Bitraf"
- board text added: "Polargraph v0.1 2022"
